File: pcb/waveshare-round-128-rpi2350-piggyback/waveshare-round-128-rpi2350-piggyback.kicad_sch (KiCad schematic)
At the start: 0 parts

Commit message: Final Rev.A PCB design.
Parts:
- added J1, J2: Conn_02x10_Odd_Even, Connector_PinHeader_1.27mm:PinHeader_2x10_P1.27mm_Vertical_SMD, symbol Connector_Generic:Conn_02x10_Odd_Even
- added TP0: 0, TestPoint:TestPoint_Pad_D2.0mm, symbol Connector:TestPoint
- added TP1: 1, TestPoint:TestPoint_Pad_D2.0mm, symbol Connector:TestPoint
- added TP10: 10 LCD CLK, TestPoint:TestPoint_Pad_D2.0mm, symbol Connector:TestPoint
- added TP11: 11 LDC MOSI, TestPoint:TestPoint_Pad_D2.0mm, symbol Connector:TestPoint
- added TP12: LCD RST 12, TestPoint:TestPoint_Pad_D2.0mm, symbol Connector:TestPoint
- added TP13: 13, TestPoint:TestPoint_Pad_D2.0mm, symbol Connector:TestPoint
- added TP14: 14, TestPoint:TestPoint_Pad_D2.0mm, symbol Connector:TestPoint
- added TP15: 15, TestPoint:TestPoint_Pad_D2.0mm, symbol Connector:TestPoint
- added TP16: 16, TestPoint:TestPoint_Pad_D2.0mm, symbol Connector:TestPoint
- added TP17: 17, TestPoint:TestPoint_Pad_D2.0mm, symbol Connector:TestPoint
- added TP18: 18, TestPoint:TestPoint_Pad_D2.0mm, symbol Connector:TestPoint
- added TP19: 19, TestPoint:TestPoint_Pad_D2.0mm, symbol Connector:TestPoint
- added TP2: 2, TestPoint:TestPoint_Pad_D2.0mm, symbol Connector:TestPoint
- added TP20: 20, TestPoint:TestPoint_Pad_D2.0mm, symbol Connector:TestPoint
- added TP21: 21, TestPoint:TestPoint_Pad_D2.0mm, symbol Connector:TestPoint
- added TP22: 22, TestPoint:TestPoint_Pad_D2.0mm, symbol Connector:TestPoint
- added TP23: IMU INT1 23, TestPoint:TestPoint_Pad_D2.0mm, symbol Connector:TestPoint
- added TP24: IMU INT2 24, TestPoint:TestPoint_Pad_D2.0mm, symbol Connector:TestPoint
- added TP25: LCD BL 25, TestPoint:TestPoint_Pad_D2.0mm, symbol Connector:TestPoint
- added TP26: 26, TestPoint:TestPoint_Pad_D2.0mm, symbol Connector:TestPoint
- added TP27: 27, TestPoint:TestPoint_Pad_D2.0mm, symbol Connector:TestPoint
- added TP28: 28, TestPoint:TestPoint_Pad_D2.0mm, symbol Connector:TestPoint
- added TP29: BAT ADC 29, TestPoint:TestPoint_Pad_D2.0mm, symbol Connector:TestPoint
- added TP3: 3, TestPoint:TestPoint_Pad_D2.0mm, symbol Connector:TestPoint
- added TP30: SW Clk, TestPoint:TestPoint_Pad_D2.0mm, symbol Connector:TestPoint
- added TP31: SW DIO, TestPoint:TestPoint_Pad_D2.0mm, symbol Connector:TestPoint
- added TP32: Boot, TestPoint:TestPoint_Pad_D2.0mm, symbol Connector:TestPoint
- added TP33: Run, TestPoint:TestPoint_Pad_D2.0mm, symbol Connector:TestPoint
- added TP34: ADC AVdd, TestPoint:TestPoint_Pad_D2.0mm, symbol Connector:TestPoint
- added TP4: 4, TestPoint:TestPoint_Pad_D2.0mm, symbol Connector:TestPoint
- added TP40, TP41: GND, TestPoint:TestPoint_Pad_D4.0mm, symbol Connector:TestPoint
- added TP42: Vsys, TestPoint:TestPoint_Pad_D2.5mm, symbol Connector:TestPoint
- added TP5: 5, TestPoint:TestPoint_Pad_D2.0mm, symbol Connector:TestPoint
- added TP6: 6 I2C SDA, TestPoint:TestPoint_Pad_D2.0mm, symbol Connector:TestPoint
- added TP7: 7 I2C SCL, TestPoint:TestPoint_Pad_D2.0mm, symbol Connector:TestPoint
- added TP8: 8 LCD CD, TestPoint:TestPoint_Pad_D2.0mm, symbol Connector:TestPoint
- added TP9: 9 LCD ~{CS}, TestPoint:TestPoint_Pad_D2.0mm, symbol Connector:TestPoint
Connections:
- new net ADC_AVDD: J2.18 (Pin_18), TP34.1
- new net BOOT: J2.16 (Pin_16), TP32.1
- new net GND: J1.19 (Pin_19), J2.19 (Pin_19), J2.20 (Pin_20), TP40.1, TP41.1
- new net GP0: J1.1 (Pin_1), TP0.1
- new net GP1: J1.3 (Pin_3), TP1.1
- new net GP10: J1.6 (Pin_6), TP10.1
- new net GP11: J1.8 (Pin_8), TP11.1
- new net GP12: J1.10 (Pin_10), TP12.1
- new net GP13: J1.12 (Pin_12), TP13.1
- new net GP14: J1.14 (Pin_14), TP14.1
- new net GP15: J1.16 (Pin_16), TP15.1
- new net GP16: J2.1 (Pin_1), TP16.1
- new net GP17: J2.3 (Pin_3), TP17.1
- new net GP18: J2.5 (Pin_5), TP18.1
- new net GP19: J2.7 (Pin_7), TP19.1
- new net GP2: J1.5 (Pin_5), TP2.1
- new net GP20: J2.9 (Pin_9), TP20.1
- new net GP21: J2.11 (Pin_11), TP21.1
- new net GP22: J2.13 (Pin_13), TP22.1
- new net GP23: J2.15 (Pin_15), TP23.1
- new net GP24: J2.2 (Pin_2), TP24.1
- new net GP25: J2.4 (Pin_4), TP25.1
- new net GP26: J2.6 (Pin_6), TP26.1
- new net GP27: J2.8 (Pin_8), TP27.1
- new net GP28: J2.10 (Pin_10), TP28.1
- new net GP29: J2.12 (Pin_12), TP29.1
- new net GP3: J1.7 (Pin_7), TP3.1
- new net GP4: J1.9 (Pin_9), TP4.1
- new net GP5: J1.11 (Pin_11), TP5.1
- new net GP6: J1.13 (Pin_13), TP6.1
- new net GP7: J1.15 (Pin_15), TP7.1
- new net GP8: J1.2 (Pin_2), TP8.1
- new net GP9: J1.4 (Pin_4), TP9.1
- new net RUN: J2.14 (Pin_14), TP33.1
- new net SWCLK: J1.18 (Pin_18), TP30.1
- new net SWDIO: J1.20 (Pin_20), TP31.1
- new net VSYS: J1.17 (Pin_17), J2.17 (Pin_17), TP42.1
Other:
- note added: "Note: J1 and J2 pin numbers are "Mirrored" relative to motherboard's pins."
- note added: "Reserved Pins"
- company: (none) -> Circuit Monkey -- Mark J Koch
- title: (none) -> Piggyback for Waveshare Round 1.28" LCD w/ RPi2350
